File: src/main_power_hub_elec/mpm_test_board/mpm_test_board.kicad_sch (KiCad schematic)
At the start: 29 parts, among them J1 Conn_01x10_Pin, J4 XT60F, J5 XT90M, J6 XT60M, Q1 SSM3K333R, Q2 SSM3K333R, Q3 SSM3K333R, Q4 Q_Dual_NPN_NPN_E1B1C2E2B2C1, Q5 IRFH7440TRPBF, SW1 E-STOP

Commit message: Improved design, Added matching ltspice sim
Parts:
- removed Q2, Q3: SSM3K333R, Package_TO_SOT_SMD:SOT-23-3, symbol Transistor_FET:Q_NMOS_GSD
- removed R12: 470k, Resistor_SMD:R_0402_1005Metric, symbol Bluesat:R_CompactH
- removed R13: 100R, Resistor_SMD:R_0402_1005Metric, symbol Bluesat:R_CompactH
- removed R20: 1k, Resistor_SMD:R_0402_1005Metric, symbol Bluesat:R_CompactH
- removed SW1: E-STOP, symbol Switch:SW_SPDT
- added J3: SM02B-PASS, Bluesat:SM02B-PASS, symbol Connector:Conn_01x02_Pin
- added unit 2 of Q4
- Q4: value Q_Dual_NPN_NPN_E1B1C2E2B2C1 -> BC846S
- R10: value 470k -> 1k
- R7: value 100R -> 10k
- R9: value 470k -> 2M2
Connections:
- net +12V: now also D6.1 (A1); no longer D6.2 (A2)
- net +3V3: now also R7.2; no longer JP1.1 (A)
- net Estop: now also R7.1, J3.1 (Pin_1), Q4.5 (B2)
- net GND: now also D3.2 (A2), D6.2 (A2), J3.2 (Pin_2), Q4.4 (E2); no longer D3.1 (A1), D6.1 (A1)
- net GateChanA: now also D9.2 (A), JP1.3 (B), Q4.6 (C1), R9.2
- net VBUS: now also D3.1 (A1); no longer D3.2 (A2), JP1.3 (B), R10.1
- net Vdrive: now also JP1.1 (A); no longer C37.2, D12.1 (K)
- net at JP1.2 (C): now also Q4.3 (C2)
- new net: C37.2, D12.1 (K), R10.1
Other:
- note added: "3v3 allows direct stm32 sensing"
- note added: "Add resistor options/jumper to tune t_fall (BJT gain)"
- note added: "Add resistor options/jumper to tune t_rise (softstart)"
- note added: "Can be either vdrive or gate. gate might be better, needs one bjt per channel but doable with dual npn"
- note added: "Charge Pump"
- note added: "Debug/for probing/input"
- note added: "If using vdrive, Q4B should be its own dedicated npn/nmos"
- note removed: "3. Charge Pump"
- note removed: "3v3 lets us sense with stm32 otherwise just use voltage divider to sense vbus (?)"
- note removed: "Add resistor options/jumper to tune t_fall"
- note removed: "Add resistor options/jumper to tune t_rise"
- note removed: "Confirm how we are going to represent the E-stop"
- note removed: "Debug/for probing"
- moved on the sheet: C23, D5, D9, J4, Q4A, Q5, R11, R6, R7, R9

Commit message: V1 of test board: routed board and slight modification to schematic
Parts:
- removed C23: 1n, Capacitor_SMD:C_0402_1005Metric, symbol Bluesat:C_CompactH
- removed D9: SBR0240LP-7, Diode_SMD:D_SOD-882D, symbol Device:D_Schottky
- added D7: SBR0240LP-7, Diode_SMD:D_SOD-882D, symbol Device:D_Schottky
- added J10: Source, Connector_PinHeader_2.54mm:PinHeader_1x01_P2.54mm_Vertical, symbol Connector:Conn_01x01_Pin
- added J11: Gate, Connector_PinHeader_2.54mm:PinHeader_1x01_P2.54mm_Vertical, symbol Connector:Conn_01x01_Pin
- added J2, J7: Conn_01x01_Pin, Connector_PinHeader_2.54mm:PinHeader_1x01_P2.54mm_Vertical, symbol Connector:Conn_01x01_Pin
- added J8: (no value), Connector_PinHeader_2.54mm:PinHeader_1x02_P2.54mm_Vertical, symbol Connector:Conn_01x02_Pin
- added J9: Conn_01x10_Pin, Connector_PinHeader_2.54mm:PinHeader_1x03_P2.54mm_Vertical, symbol Connector:Conn_01x03_Pin
- added R12: 10k, Resistor_SMD:R_0402_1005Metric, symbol Bluesat:R_CompactH
- J1: footprint (none) -> Connector_PinHeader_2.54mm:PinHeader_1x10_P2.54mm_Vertical; now not fitted
- J6: value XT60M -> (none); footprint Connector_AMASS:AMASS_XT60PW-M_1x02_P7.20mm_Horizontal -> Connector_PinHeader_2.54mm:PinHeader_1x01_P2.54mm_Vertical; symbol Connector:Conn_01x02_Pin -> Connector:Conn_01x01_Pin
- JP1: footprint (none) -> Jumper:SolderJumper-3_P1.3mm_Open_Pad1.0x1.5mm_NumberLabels
Connections:
- net +12V: now also J6.1 (Pin_1); no longer J6.2 (Pin_2)
- net +3V3: now also J7.1 (Pin_1), J8.2 (Pin_2)
- net CLK_IN: now also J2.1 (Pin_1)
- net DisableChanA: now also J8.1 (Pin_1), R12.2
- net GND: now also J9.1 (Pin_1), J9.2 (Pin_2), J9.3 (Pin_3), R12.1; no longer J6.1 (Pin_1)
- net GateChanA: now also D7.2 (A), J11.1 (Pin_1)
- net SourceChanA: now also J10.1 (Pin_1)
- net Vdrive: now also D7.1 (K)
Other:
- note added: "3.3V"
- note removed: "Do we add 3v3 regulator or input?"
- note removed: "Use button to represent STM32 (?) Also allow external input"
- moved on the sheet: R9
