Commit message: Get the BESCs working (maybe)

File: src/rover/description/core/ros2control.xacro (robot description, xacro)
@@ -2,13 +2,14 @@
 <robot xmlns:xacro="http://www.ros.org/wiki/xacro">
     <!-- Specify the joints that are in a single swerve module, limits are specified in joint declaration! -->
-    <xacro:macro name="ros2control_swerve_drive_iface" params="name subject_id">
+    <xacro:macro name="ros2control_swerve_drive_iface" params="name device_id">
         <joint name="db_${name}_fork_tyre_joint">
+            <param name="device_id">${device_id}</param>
             <command_interface name="velocity">
                 <limits enable="true"/>
-                <param name="subject_id">${subject_id}</param>
             </command_interface>
+            <state_interface name="velocity"/>
         </joint>
     </xacro:macro>
-    <xacro:macro name="ros2control_swerve_turn_iface" params="name subject_id">
+    <xacro:macro name="ros2control_swerve_turn_iface" params="name device_id">
         <joint name="db_${name}_smount_fork_joint">
             <command_interface name="position">
@@ -25,11 +26,11 @@
         <hardware>
             <plugin>cyphal_vesc_driver/CyphalVescDriver</plugin>
-            <param name="canbus">can-all</param>
-            <param name="nodeid">69</param>
+            <param name="can_bus">can-all</param>
+            <param name="node_id">69</param>
         </hardware>
-        <xacro:ros2control_swerve_drive_iface name="fl" subject_id="3050"/>
-        <xacro:ros2control_swerve_drive_iface name="fr" subject_id="3060"/>
-        <xacro:ros2control_swerve_drive_iface name="bl" subject_id="3070"/>
-        <xacro:ros2control_swerve_drive_iface name="br" subject_id="3080"/>
+        <xacro:ros2control_swerve_drive_iface name="fl" device_id="3050"/>
+        <xacro:ros2control_swerve_drive_iface name="fr" device_id="3060"/>
+        <xacro:ros2control_swerve_drive_iface name="bl" device_id="3070"/>
+        <xacro:ros2control_swerve_drive_iface name="br" device_id="3080"/>
     </ros2_control>
     <ros2_control name="MockComponents" type="system">
@@ -37,8 +38,8 @@
             <plugin>mock_components/GenericSystem</plugin>
         </hardware>
-        <xacro:ros2control_swerve_turn_iface name="fl" subject_id="3000"/>
-        <xacro:ros2control_swerve_turn_iface name="fr" subject_id="3010"/>
-        <xacro:ros2control_swerve_turn_iface name="bl" subject_id="3020"/>
-        <xacro:ros2control_swerve_turn_iface name="br" subject_id="3030"/>
+        <xacro:ros2control_swerve_turn_iface name="fl" device_id="3000"/>
+        <xacro:ros2control_swerve_turn_iface name="fr" device_id="3010"/>
+        <xacro:ros2control_swerve_turn_iface name="bl" device_id="3020"/>
+        <xacro:ros2control_swerve_turn_iface name="br" device_id="3030"/>
         <xacro:ros2control_drivebase_suspension_pivot side="l"/>
         <xacro:ros2control_drivebase_suspension_pivot side="r"/>

Commit message: Get the BESCs working fr

File: src/rover/description/core/ros2control.xacro (robot description, xacro)
@@ -2,7 +2,8 @@
 <robot xmlns:xacro="http://www.ros.org/wiki/xacro">
     <!-- Specify the joints that are in a single swerve module, limits are specified in joint declaration! -->
-    <xacro:macro name="ros2control_swerve_drive_iface" params="name device_id">
+    <xacro:macro name="ros2control_swerve_drive_iface" params="name device_id invert">
         <joint name="db_${name}_fork_tyre_joint">
             <param name="device_id">${device_id}</param>
+            <param name="invert">${invert}</param>
             <command_interface name="velocity">
                 <limits enable="true"/>
@@ -26,11 +27,11 @@
         <hardware>
             <plugin>cyphal_vesc_driver/CyphalVescDriver</plugin>
-            <param name="can_bus">can-all</param>
+            <param name="can_bus">can-vesc</param>
             <param name="node_id">69</param>
         </hardware>
-        <xacro:ros2control_swerve_drive_iface name="fl" device_id="3050"/>
-        <xacro:ros2control_swerve_drive_iface name="fr" device_id="3060"/>
-        <xacro:ros2control_swerve_drive_iface name="bl" device_id="3070"/>
-        <xacro:ros2control_swerve_drive_iface name="br" device_id="3080"/>
+        <xacro:ros2control_swerve_drive_iface name="fl" device_id="3050" invert="false"/>
+        <xacro:ros2control_swerve_drive_iface name="fr" device_id="3060" invert="true"/>
+        <xacro:ros2control_swerve_drive_iface name="bl" device_id="3070" invert="false"/>
+        <xacro:ros2control_swerve_drive_iface name="br" device_id="3080" invert="true"/>
     </ros2_control>
     <ros2_control name="MockComponents" type="system">

Commit message: 221 besc driver (#207)
* Add architectural information for initial design of BESC ros2_control hardware interface

* Add architectural description for FFI Rust/C++ Canadensis layer

* start rust and write data parts in cpp

* on init code

* on init code

* on_init written

* Implement remaining BESC hardware interface Rust FFI API

* Add podman instructions for broken images </3

* generated bridge

* Write a draft of the Rust side of the BESC driver

* remove old files

* Remove some duplicate changes from main (diff. paths)

* Move rust/uv setup after USER statement to install them properly

* Get skill issued by CMake

* I understand now

* Builds

* Builds and crashes & init, add more checks / params

* Actually link smiley

* Make Rust aware of device names as it is slightly cleaner

* Get the BESCs working (maybe)

* Get the BESCs working fr

* Fix install nvim script to not fuck cargo/uv

* For the goy

* Update xacro

* Fix the cpp bus driver

* oops

* state

* Baka

* Stuff

---------

Co-authored-by: fox-58 <sophie@foxy.net.au>
Co-authored-by: Evan La Fontaine <navelafontaine@gmail.com>
Co-authored-by: Aavin Fernando <aavin.fernando@gmail.com>

File: src/rover/description/core/ros2control.xacro (robot description, xacro)
@@ -2,17 +2,23 @@
 <robot xmlns:xacro="http://www.ros.org/wiki/xacro">
     <!-- Specify the joints that are in a single swerve module, limits are specified in joint declaration! -->
-    <xacro:macro name="ros2control_swerve_drive_iface" params="name subject_id">
+    <xacro:macro name="ros2control_swerve_drive_iface" params="name device_id invert">
         <joint name="db_${name}_fork_tyre_joint">
+            <param name="device_id">${device_id}</param>
+            <param name="invert">${invert}</param>
+            <param name="type">besc</param>
             <command_interface name="velocity">
                 <limits enable="true"/>
-                <param name="subject_id">${subject_id}</param>
             </command_interface>
+            <state_interface name="velocity"/>
         </joint>
     </xacro:macro>
-    <xacro:macro name="ros2control_swerve_turn_iface" params="name subject_id">
+    <xacro:macro name="ros2control_swerve_turn_iface" params="name device_id">
         <joint name="db_${name}_smount_fork_joint">
+            <param name="device_id">${device_id}</param>
+            <param name="type">stepper</param>
             <command_interface name="position">
                 <limits enable="true"/>
             </command_interface>
+            <state_interface name="position"/>
         </joint>
     </xacro:macro>
@@ -22,12 +28,18 @@
         </joint>
     </xacro:macro>
-    <ros2_control name="VESCControlSystem" type="system">
+    <ros2_control name="CoreControlSystem" type="system">
         <hardware>
-            <plugin>cyphal_vesc_driver/CyphalVescDriver</plugin>
+            <plugin>cyphal_bus_driver/CyphalBusDriver</plugin>
+            <param name="can_bus">can-all</param>
+            <param name="node_id">69</param>
         </hardware>
-        <xacro:ros2control_swerve_drive_iface name="fl" subject_id="3050"/>
-        <xacro:ros2control_swerve_drive_iface name="fr" subject_id="3060"/>
-        <xacro:ros2control_swerve_drive_iface name="bl" subject_id="3070"/>
-        <xacro:ros2control_swerve_drive_iface name="br" subject_id="3080"/>
+        <xacro:ros2control_swerve_drive_iface name="fl" device_id="3050" invert="false"/>
+        <xacro:ros2control_swerve_drive_iface name="fr" device_id="3060" invert="true"/>
+        <xacro:ros2control_swerve_drive_iface name="bl" device_id="3070" invert="false"/>
+        <xacro:ros2control_swerve_drive_iface name="br" device_id="3080" invert="true"/>
+        <xacro:ros2control_swerve_turn_iface name="fl" device_id="3000"/>
+        <xacro:ros2control_swerve_turn_iface name="fr" device_id="3010"/>
+        <xacro:ros2control_swerve_turn_iface name="bl" device_id="3020"/>
+        <xacro:ros2control_swerve_turn_iface name="br" device_id="3030"/>
     </ros2_control>
     <ros2_control name="MockComponents" type="system">
@@ -35,8 +47,4 @@
             <plugin>mock_components/GenericSystem</plugin>
         </hardware>
-        <xacro:ros2control_swerve_turn_iface name="fl" subject_id="3000"/>
-        <xacro:ros2control_swerve_turn_iface name="fr" subject_id="3010"/>
-        <xacro:ros2control_swerve_turn_iface name="bl" subject_id="3020"/>
-        <xacro:ros2control_swerve_turn_iface name="br" subject_id="3030"/>
         <xacro:ros2control_drivebase_suspension_pivot side="l"/>
         <xacro:ros2control_drivebase_suspension_pivot side="r"/>
