File: src/besc_elec/mosfets.kicad_sch (KiCad schematic)
At the start: 12 parts, among them Q301 IRFH7440TRPBF, Q302 IRFH7440TRPBF

Commit message: added DRV8323HRTAR symbol and footprint
Parts:
- added C302: 1n, symbol Bluesat:C_CompactV
- added R308: 47k, symbol Bluesat:R_CompactV
- added R309: 4k7, symbol Bluesat:R_CompactV
Connections:
- net GND: now also C302.1, R309.2
- net PHASE: now also R308.1
- net LOW renamed SENS
- new net PHS_SENS: C302.2, R308.2, R309.1
Other:
- note added: "<- two close to MCU"

Commit message: switched gate driver variant from RS->HR
Parts:
- renumbered C302 to C304
Changed lines of the file:
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@@
 				)
 				(path "/2059a583-03d9-42e7-b042-844898d8f177/395e1093-67ec-4614-b25c-b37e14ae8318"
-					(reference "R2")
-					(unit 1)
-				)
-				(path "/2059a583-03d9-42e7-b042-844898d8f177/43e157cb-6b50-47c8-9e44-0b1971389d5f"
-					(reference "R3")
+					(reference "R409")
+					(unit 1)
+				)
+				(path "/2059a583-03d9-42e7-b042-844898d8f177/43e157cb-6b50-47c8-9e44-0b1971389d5f"
+					(reference "R509")
 					(unit 1)
 				)
@@
 				)
 				(path "/2059a583-03d9-42e7-b042-844898d8f177/395e1093-67ec-4614-b25c-b37e14ae8318"
-					(reference "R5")
-					(unit 1)
-				)
-				(path "/2059a583-03d9-42e7-b042-844898d8f177/43e157cb-6b50-47c8-9e44-0b1971389d5f"
-					(reference "R6")
+					(reference "R408")
+					(unit 1)
+				)
+				(path "/2059a583-03d9-42e7-b042-844898d8f177/43e157cb-6b50-47c8-9e44-0b1971389d5f"
+					(reference "R508")
 					(unit 1)
 				)
@@
 		(dnp no)
 		(fields_autoplaced yes)
-		(property "Reference" "C302"
+		(property "Reference" "C304"
 			(at 178.181 107.188 90)
 			(show_name no)
@@
 			(project "vesc2"
 				(path "/2059a583-03d9-42e7-b042-844898d8f177/1b823304-293f-4595-a426-e06902eaf0d9"
-					(reference "C302")
-					(unit 1)
-				)
-				(path "/2059a583-03d9-42e7-b042-844898d8f177/395e1093-67ec-4614-b25c-b37e14ae8318"
-					(reference "C2")
-					(unit 1)
-				)
-				(path "/2059a583-03d9-42e7-b042-844898d8f177/43e157cb-6b50-47c8-9e44-0b1971389d5f"
-					(reference "C3")
-					(unit 1)
-				)
+					(reference "C304")
+					(unit 1)
+				)
+				(path "/2059a583-03d9-42e7-b042-844898d8f177/395e1093-67ec-4614-b25c-b37e14ae8318"
+					(reference "C404")
+					(unit 1)
+				)
+				(path "/2059a583-03d9-42e7-b042-844898d8f177/43e157cb-6b50-47c8-9e44-0b1971389d5f"
+					(reference "C504")
+					(unit 1)
+				)
