File: src/debug_adapter_elec/debug_adapter/debug_adapter.kicad_pcb (KiCad board)
At the start: 2 copper layers, 34 x 16 mm, 9 parts, among them J1 Conn_02x03_Odd_Even, J2 Conn_02x05_Odd_Even, J3 Conn_01x10

Commit message: minor changes
Other:
- board text added: "By Saksham Gulati :)"
- board text removed: "By Saksham Gulati"
Changed lines of the file:
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@@
 		(layer "Edge.Cuts")
 	)
-	(gr_text "By Saksham Gulati"
+	(gr_text "By Saksham Gulati :)"
 		(at 102.5 109.5 0)
 		(layer "B.SilkS")

Commit message: debug adapter design v2
Parts:
- removed TP1, TP2, TP3, TP4, TP5, TP6: TestPoint, TestPoint:TestPoint_Pad_D2.0mm
- added 3V3: TestPoint, TestPoint:TestPoint_Pad_D2.0mm, B.Cu at (145.4, 103.0)
- added GND: TestPoint, TestPoint:TestPoint_Pad_D2.0mm, B.Cu at (156.4, 103.0)
- added NRST: TestPoint, TestPoint:TestPoint_Pad_D2.0mm, B.Cu at (145.4, 99.3)
- added SWCLK: TestPoint, TestPoint:TestPoint_Pad_D2.0mm, B.Cu at (145.4, 106.8)
- added SWDIO: TestPoint, TestPoint:TestPoint_Pad_D2.0mm, B.Cu at (156.4, 106.8)
- added SWO: TestPoint, TestPoint:TestPoint_Pad_D2.0mm, B.Cu at (156.4, 99.3)
- J1: footprint easyeda2kicad:CONN-TH_215570-6 -> Bluesat:IDC6; moved to B.Cu
- moved J2 65.7 mm to (138.1, 98.0)
- moved J1 65.2 mm to (150.9, 103.0), turned to -90 degrees
- moved J3 57.9 mm to (156.4, 103.0)
Connections:
- J2 pad 1: /SWDIO -> /SWCLK
- J2 pad 10: /5V -> unconnected-(J2-Pin_10-Pad10)
- J2 pad 3: /GND -> /SWDIO
- J2 pad 4: /GND -> unconnected-(J2-Pin_4-Pad4)
- J2 pad 5: /SWCLK -> /GND
- J2 pad 6: /SWIM -> /GND
- J2 pad 7: /3V3 -> unconnected-(J2-Pin_7-Pad7)
- J2 pad 8: /3V3 -> unconnected-(J2-Pin_8-Pad8)
- J2 pad 9: /5V -> unconnected-(J2-Pin_9-Pad9)
- J3 pad 1: /3V3 -> unconnected-(J3-Pin_1-Pad1)
- J3 pad 10: /5V -> unconnected-(J3-Pin_10-Pad10)
- J3 pad 7: /TXD -> unconnected-(J3-Pin_7-Pad7)
- J3 pad 8: /RXD -> unconnected-(J3-Pin_8-Pad8)
Routing:
- net /GND: track 36.4 -> 11.6 mm, vias 1 -> 2
- net /SWCLK: track 38.8 -> 24.1 mm, vias 0 -> 1
- net /NRST: track 30.4 -> 16.0 mm, vias 0 -> 1
- net /3V3: track 16.4 -> 3.48 mm
- net /SWDIO: track 35.7 -> 24.8 mm, vias 1 -> 2
- net /SWO: track 19.1 -> 11.2 mm
- added copper zone on B.Cu, net /GND
Other:
- board size 34 x 16 mm -> 23.6 x 14 mm
- board text added: ":)"
- board text added: "By Saksham Gulati"
- board text added: "Debug Adapter"
- board text added: "R1P0"
- board text removed: "By Saksham Gulati :)"

Commit message: minor changes
Routing:
- net /GND: track 11.6 -> 9.04 mm
Changed lines of the file:
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@@
 		(sheetname "/")
 		(sheetfile "debug_adapter.kicad_sch")
-		(units
-			(unit
-				(name "A")
-				(pins "1" "3" "5" "7" "9" "2" "4" "6" "8" "10")
-			)
-		)
 		(attr through_hole)
 		(duplicate_pad_numbers_are_jumpers no)
@@
 				(type solid)
 			)
+			(layer "F.SilkS")
+		)
+		(fp_rect
+			(start 3.92 2.5)
+			(end 4.21 7.75)
+			(stroke
+				(width 0.12)
+				(type solid)
+			)
+			(fill yes)
 			(layer "F.SilkS")
 		)
@@
 	)
 	(segment
-		(start 138.105 103.1)
-		(end 140.645 103.1)
-		(width 1)
-		(layer "B.Cu")
-		(net "/GND")
-	)
-	(segment
 		(start 154.395 103.52)
 		(end 151.145 103.52)
@@
 		(name "GND")
 		(hatch edge 0.5)
-		(connect_pads
+		(connect_pads yes
 			(clearance 0.5)
 		)
