File: src/debug_adapter_elec/debug_adapter/debug_adapter.kicad_sch (KiCad schematic)
At the start: 9 parts, among them J1 Conn_02x03_Odd_Even, J2 Conn_02x05_Odd_Even, J3 Conn_01x10

Commit message: debug adapter design v2
Parts:
- J1: footprint easyeda2kicad:CONN-TH_215570-6 -> Bluesat:IDC6
- renumbered TP4 to 3V3, TP3 to GND1, TP2 to NRST1, TP6 to SWCLK1, TP5 to SWDIO1, TP1 to SWO1
Connections:
- net 3V3: no longer J2.7 (Pin_7), J2.8 (Pin_8), J3.1 (Pin_1)
- net 5V: no longer J2.10 (Pin_10), J2.9 (Pin_9), J3.10 (Pin_10)
- net GND: now also J2.5 (Pin_5), J2.6 (Pin_6); no longer J2.3 (Pin_3), J2.4 (Pin_4)
- net RXD: no longer J3.8 (Pin_8)
- net SWCLK: now also J2.1 (Pin_1); no longer J2.5 (Pin_5)
- net SWDIO: now also J2.3 (Pin_3); no longer J2.1 (Pin_1)
- net SWIM: no longer J2.6 (Pin_6)
- net TXD: no longer J3.7 (Pin_7)
- no-connect marks 8 -> 9
Other:
- note added: "- 3V3 not connected since clones don't sense 3V3. - 5V not connected since its not passed to device under test - V3 UART pins and V2 SWIM pin not connected since its not passed to device under test."
- note added: "2x5 Keyed Duponts to STLink V2 clone"
- note added: "Crimped IDC6 to device under test"
- note removed: "- 3V3 not connected on V2 since V2 supplies (not senses) 3V3. - 5V not connected since its not passed to device under test - V3 UART pins and V2 SWIM pin not connected since its not passed to device under test."
- note removed: "2x5 Keyed Duponts to STLink V2"
- note removed: "[Connector] to DUT"

Commit message: minor changes
Other:
- note added: "3V3"
- note added: "5V"
- note added: "RXD"
- note added: "SWIM"
- note added: "TXD"
Changed lines of the file:
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@@
 	(generator_version "10.0")
 	(paper "A4")
+	(text "3V3"
+		(exclude_from_sim no)
+		(at 48.514 177.292 0)
+		(effects
+			(font
+				(size 1.27 1.27)
+			)
+			(justify right)
+		)
+	)
 	(text "10 JST SH to\nSTLink V3 clone"
 		(exclude_from_sim no)
@@
 		)
 	)
+	(text "5V"
+		(exclude_from_sim no)
+		(at 48.26 179.832 0)
+		(effects
+			(font
+				(size 1.27 1.27)
+			)
+			(justify right)
+		)
+	)
+	(text "SWIM"
+		(exclude_from_sim no)
+		(at 48.514 171.958 0)
+		(effects
+			(font
+				(size 1.27 1.27)
+			)
+			(justify right)
+		)
+	)
+	(text "3V3"
+		(exclude_from_sim no)
+		(at 92.964 181.61 90)
+		(effects
+			(font
+				(size 1.27 1.27)
+			)
+			(justify left)
+		)
+	)
 	(text "2x5 Keyed Duponts\nto STLink V2 clone"
 		(exclude_from_sim no)
@@
 		)
 	)
+	(text "5V"
+		(exclude_from_sim no)
+		(at 70.612 181.61 90)
+		(effects
+			(font
+				(size 1.27 1.27)
+			)
+			(justify left)
+		)
+	)
+	(text "5V"
+		(exclude_from_sim no)
+		(at 23.114 180.086 0)
+		(effects
+			(font
+				(size 1.27 1.27)
+			)
+			(justify left)
+		)
+	)
+	(text "TXD\n"
+		(exclude_from_sim no)
+		(at 77.724 181.864 90)
+		(effects
+			(font
+				(size 1.27 1.27)
+			)
+			(justify left)
+		)
+	)
+	(text "3V3"
+		(exclude_from_sim no)
+		(at 23.114 177.292 0)
+		(effects
+			(font
+				(size 1.27 1.27)
+			)
+			(justify left)
+		)
+	)
+	(text "RXD"
+		(exclude_from_sim no)
+		(at 75.184 181.864 90)
+		(effects
+			(font
+				(size 1.27 1.27)
+			)
+			(justify left)
+		)
+	)
 	(no_connect
 		(at 71.12 175.26)
@@
 	(wire
 		(pts
-			(xy 71.12 177.8) (xy 71.12 181.61)
-		)
-		(stroke
-			(width 0)
-			(type default)
-		)
-	)
-	(wire
-		(pts
 			(xy 144.78 172.72) (xy 152.4 172.72)
 		)
@@
 	(wire
 		(pts
-			(xy 44.45 172.72) (xy 48.26 172.72)
-		)
-		(stroke
-			(width 0)
-			(type default)
-		)
-	)
-	(wire
-		(pts
 			(xy 124.46 172.72) (xy 132.08 172.72)
 		)
@@
 	(wire
 		(pts
-			(xy 78.74 177.8) (xy 78.74 181.61)
-		)
-		(stroke
-			(width 0)
-			(type default)
-		)
-	)
-	(wire
-		(pts
 			(xy 86.36 181.61) (xy 86.36 175.26)
 		)
@@
 	(wire
 		(pts
-			(xy 76.2 177.8) (xy 76.2 181.61)
-		)
-		(stroke
-			(width 0)
-			(type default)
-		)
-	)
-	(wire
-		(pts
-			(xy 44.45 177.8) (xy 48.26 177.8)
-		)
-		(stroke
-			(width 0)
-			(type default)
-		)
-	)
-	(wire
-		(pts
-			(xy 22.86 180.34) (xy 26.67 180.34)
-		)
-		(stroke
-			(width 0)
-			(type default)
-		)
-	)
-	(wire
-		(pts
 			(xy 81.28 181.61) (xy 81.28 175.26)
 		)
@@
 	(wire
 		(pts
-			(xy 22.86 177.8) (xy 26.67 177.8)
-		)
-		(stroke
-			(width 0)
-			(type default)
-		)
-	)
-	(wire
-		(pts
-			(xy 93.98 177.8) (xy 93.98 181.61)
-		)
-		(stroke
-			(width 0)
-			(type default)
-		)
-	)
-	(wire
-		(pts
 			(xy 144.78 175.26) (xy 152.4 175.26)
-		)
-		(stroke
-			(width 0)
-			(type default)
-		)
-	)
-	(wire
-		(pts
-			(xy 44.45 180.34) (xy 48.26 180.34)
 		)
 		(stroke
@@
 		)
 	)
-	(label "TXD"
-		(at 78.74 181.61 90)
-		(effects
-			(font
-				(size 1.27 1.27)
-			)
-			(justify left bottom)
-		)
-	)
-	(label "3V3"
-		(at 93.98 181.61 90)
-		(effects
-			(font
-				(size 1.27 1.27)
-			)
-			(justify left bottom)
-		)
-	)
-	(label "3V3"
-		(at 48.26 177.8 180)
-		(effects
-			(font
-				(size 1.27 1.27)
-			)
-			(justify right bottom)
-		)
-	)
 	(label "NRST"
 		(at 81.28 181.61 90)
@@
 		)
 	)
-	(label "5V"
-		(at 48.26 180.34 180)
-		(effects
-			(font
-				(size 1.27 1.27)
-			)
-			(justify right bottom)
-		)
-	)
 	(label "SWCLK"
 		(at 22.86 170.18 0)
@@
 		)
 	)
-	(label "5V"
-		(at 71.12 181.61 90)
-		(effects
-			(font
-				(size 1.27 1.27)
-			)
-			(justify left bottom)
-		)
-	)
 	(label "3V3"
 		(at 152.4 172.72 180)
@@
 		)
 	)
-	(label "SWIM"
-		(at 48.26 172.72 180)
-		(effects
-			(font
-				(size 1.27 1.27)
-			)
-			(justify right bottom)
-		)
-	)
-	(label "3V3"
-		(at 22.86 177.8 0)
-		(effects
-			(font
-				(size 1.27 1.27)
-			)
-			(justify left bottom)
-		)
-	)
 	(label "SWCLK"
 		(at 88.9 181.61 90)
@@
 		)
 	)
-	(label "RXD"
-		(at 76.2 181.61 90)
-		(effects
-			(font
-				(size 1.27 1.27)
-			)
-			(justify left bottom)
-		)
-	)
 	(label "GND"
 		(at 86.36 181.61 90)
@@
 		(effects
 			(font
-				(size 1.27 1.27)
-			)
-			(justify left bottom)
-		)
-	)
-	(label "5V"
-		(at 22.86 180.34 0)
-		(effects
-			(font
